Commit message: reworked visuals for xarm6

File: data/xarm6/xarm6.urdf (robot description, URDF)
Before this commit: robot xarm6, 9 links, 8 joints
Links:
- link link1: geometry collision mesh filename=collision/link1.stl; visual mesh filename=visual/link1.dae
- link link2: geometry collision mesh filename=collision/link2.stl; visual mesh filename=visual/link2.dae
- link link3: geometry collision mesh filename=collision/link3.stl; visual mesh filename=visual/link3.dae
- link link4: geometry collision mesh filename=collision/link4.stl; visual mesh filename=visual/link4.dae
- link link5: geometry collision mesh filename=collision/link5.stl; visual mesh filename=visual/link5.dae
- link link6: geometry collision mesh filename=collision/link6.stl; visual mesh filename=visual/link6.dae
- link link_base: geometry collision mesh filename=collision/base.stl; visual mesh filename=visual/base.dae
